File: 21mtc/21mtc.kicad_pcb (KiCad board)
At the start: 2 copper layers, 48 x 24 mm, 6 parts, among them P101 CONN_01X06, P102 CONN_02X11, P103 CONN_01X11, P104 CONN_02X04, P105 CONN_01X04

Commit message: MTC21 Updates
Parts:
- added Q101: NTJD4401N, Housings_SOT-23_SOT-143_TSOT-6:SC-70-6_Handsoldering, F.Cu at (181.0, 116.0)
- added R101: R, Resistors_SMD:R_0805_HandSoldering, F.Cu at (176.0, 113.0)
- added R102: R, Resistors_SMD:R_0805_HandSoldering, F.Cu at (172.0, 112.0)
- added R103: R, Resistors_SMD:R_0805_HandSoldering, F.Cu at (169.7, 117.0)
- added R104: R, Resistors_SMD:R_0805_HandSoldering, F.Cu at (176.0, 118.0)
Connections:
- net /GND renamed GND
- P101 pad 4: /Aux4 -> Net-(P101-Pad4)
- P102 pad 20: /Aux3 -> /Aux3_ttl
- P102 pad 7: /Aux4 -> /Aux4_ttl
- P103 pad 2: /Aux3 -> Net-(P103-Pad2)
Routing:
- net Net-(P101-Pad4): track 0.00 -> 57.5 mm, vias 0 -> 2
- net Net-(P103-Pad2): track 0.00 -> 57.5 mm, vias 0 -> 2
- net /Aux3_ttl: track 0.00 -> 23.0 mm, vias 0 -> 2
- net /Aux4: track 22.8 -> 0.00 mm
- net GND: track 32.8 -> 45.4 mm
- net Net-(Q101-Pad5): track 0.00 -> 9.08 mm
- net /Aux3: track 8.63 -> 0.00 mm
- net /Aux4_ttl: track 0.00 -> 4.54 mm
- net /TrackL: track 43.5 -> 47.6 mm
- net /Motor1: track 59.6 -> 60.8 mm

Commit message: Made the design rule for power nets, track width 0.6mm
Routing:
- net Net-(P103-Pad2): track 57.5 -> 54.2 mm
- net /Aux3_ttl: track 23.0 -> 26.2 mm
- net Net-(P101-Pad4): track 57.5 -> 60.0 mm
- net /Aux4_ttl: track 4.54 -> 2.06 mm
Other:
- net class Power added: clearance 0.2, trace_width 0.6, via_dia 0.6, via_drill 0.4
Changed lines of the file:
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@@
-(kicad_pcb (version 4) (host pcbnew 4.0.0-rc2-1-stable)
+(kicad_pcb (version 4) (host pcbnew 4.0.5)
   (general
     (links 39)
-    (no_connects 11)
-    (area 139.239867 99.1342 189.100001 139.175001)
+    (no_connects 7)
+    (area 139.314867 99.2842 189.100001 127.664533)
     (thickness 1.6)
     (drawings 10)
@@
     (add_net /Hall2)
     (add_net /Hall3)
-    (add_net /Motor1)
-    (add_net /Motor2)
-    (add_net /Motor3)
     (add_net /Plus)
     (add_net /Speak1)
@@
     (add_net /TBClock)
     (add_net /TBData)
+    (add_net "Net-(P101-Pad4)")
+    (add_net "Net-(P103-Pad2)")
+    (add_net "Net-(Q101-Pad2)")
+    (add_net "Net-(Q101-Pad5)")
+  )
+  (net_class Power ""
+    (clearance 0.2)
+    (trace_width 0.6)
+    (via_dia 0.6)
+    (via_drill 0.4)
+    (uvia_dia 0.3)
+    (uvia_drill 0.1)
+    (add_net /Motor1)
+    (add_net /Motor2)
+    (add_net /Motor3)
     (add_net /TrackL)
     (add_net /TrackR)
     (add_net /Vcc)
     (add_net GND)
-    (add_net "Net-(P101-Pad4)")
-    (add_net "Net-(P103-Pad2)")
-    (add_net "Net-(Q101-Pad2)")
-    (add_net "Net-(Q101-Pad5)")
   )
   (module Other:21MTC_decoder_outline (layer F.Cu)
@@
   (segment (start 150.261101 105.698599) (end 146.741099 105.698599) (width 0.25) (layer F.Cu) (net 19))
   (segment (start 150.326101 105.763599) (end 150.261101 105.698599) (width 0.25) (layer F.Cu) (net 19))
+  (segment (start 150.326101 108.238599) (end 150.326101 105.763599) (width 0.25) (layer F.Cu) (net 19))
   (segment (start 171.725001 111.089999) (end 171.660001 111.024999) (width 0.25) (layer F.Cu) (net 20))
   (segment (start 178.9938 122.1312) (end 177.7438 120.8812) (width 0.25) (layer F.Cu) (net 20))
@@
   (segment (start 149.7511 108.8136) (end 150.326101 108.238599) (width 0.25) (layer F.Cu) (net 21))
   (segment (start 148.5011 108.8136) (end 149.7511 108.8136) (width 0.25) (layer F.Cu) (net 21))
-  (segment (start 150.326101 108.238599) (end 150.326101 105.763599) (width 0.25) (layer F.Cu) (net 21))
   (segment (start 155 117) (end 152.8375 117) (width 0.25) (layer F.Cu) (net 22))
   (segment (start 152.8375 117) (end 152.7711 116.9336) (width 0.25) (layer F.Cu) (net 22))
@@
   (segment (start 154.596101 118.608899) (end 154.596101 117.008601) (width 0.25) (layer F.Cu) (net 22))
   (segment (start 154.0211 116.4336) (end 152.7711 116.4336) (width 0.25) (layer F.Cu) (net 22))
+  (segment (start 152.3238 120.8812) (end 154.596101 118.608899) (width 0.25) (layer F.Cu) (net 22))
   (segment (start 188 117) (end 186.300608 115.300608) (width 0.25) (layer B.Cu) (net 23))
   (via (at 182.33096 115.300608) (size 0.6) (drill 0.4) (layers F.Cu B.Cu) (net 23))
@@
   (segment (start 152.3238 124.3812) (end 153.9426 126) (width 0.25) (layer F.Cu) (net 23))
   (segment (start 152.3238 122.6312) (end 152.3238 120.8812) (width 0.25) (layer F.Cu) (net 23))
-  (segment (start 152.3238 120.8812) (end 154.596101 118.608899) (width 0.25) (layer F.Cu) (net 23))
   (segment (start 176 116.65) (end 176.9 116.65) (width 0.25) (layer F.Cu) (net 25))
   (segment (start 176.9 116.65) (end 177.55 116) (width 0.25) (layer F.Cu) (net 25))

Commit message: Library management
Parts:
- added G***: LOGO, 21mtc:21mtc_logo_scaled_01, F.Cu at (175.6, 116.8)
- added REF**: MountingHole_2.2mm_M2, Mounting_Holes:MountingHole_2.2mm_M2, F.Cu at (176.0, 112.1)
- moved R103 12.4 mm to (181.8, 119.3)
- moved R101 11.4 mm to (187.4, 113.3)
- moved R102 10.9 mm to (181.8, 116.8)
- moved R104 10.4 mm to (185.3, 113.3)
- moved Q101 6.54 mm to (187.1, 118.4), turned to 180 degrees
Connections:
- P101 pad 4: Net-(P101-Pad4) -> /Plus
- P101 pad 5: /TBClock -> /F0_r_y
- P101 pad 6: /TBData -> /F0_f_w
- P102 pad 12: /Motor3 -> /Aux5
- P103 pad 10: /TrackL -> Net-(P103-Pad10)
- P103 pad 11: /TrackR -> Net-(P103-Pad11)
- P103 pad 2: Net-(P103-Pad2) -> /Aux5
- P103 pad 5: /Plus -> /Motor2
- P103 pad 6: /Motor3 -> /Motor1
- P103 pad 7: /Motor2 -> /TrackL
- P103 pad 8: /Motor1 -> /TrackR
- P105 pad 1: /F0_r_y -> /TBClock
- P105 pad 2: /F0_f_w -> /TBData
- Q101 pad 3: Net-(P103-Pad2) -> Net-(P103-Pad10)
- Q101 pad 6: Net-(P101-Pad4) -> Net-(P103-Pad11)
Routing:
- net Net-(P101-Pad4): track 60.0 -> 0.00 mm, vias 2 -> 0
- net Net-(P103-Pad2): track 54.2 -> 0.00 mm, vias 2 -> 0
- net /TBData: track 48.0 -> 6.54 mm, vias 0 -> 1
- net /Aux4_ttl: track 2.06 -> 37.3 mm, vias 0 -> 2
- net /TBClock: track 33.8 -> 5.90 mm, vias 0 -> 1
- net /Aux5: track 0.00 -> 23.5 mm
- net /Motor3: track 20.2 -> 0.00 mm
- net GND: track 45.4 -> 62.3 mm, vias 2 -> 0
- net Net-(Q101-Pad2): track 0.00 -> 13.0 mm
- net /TrackR: track 51.3 -> 62.9 mm, vias 2 -> 1
- net /Motor1: track 60.8 -> 49.6 mm
- net /F0_r_y: track 39.1 -> 49.7 mm, vias 2 -> 1
- net Net-(P103-Pad10): track 0.00 -> 9.70 mm, vias 0 -> 2
- net /F0_f_w: track 42.3 -> 51.9 mm
- net /TrackL: track 47.6 -> 40.5 mm, vias 3 -> 2
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- added copper zone on F.Cu, net GND
