File: stationary/decoderinterface.kicad_pcb (KiCad board)
At the start: 2 copper layers, 50 x 50 mm, 43 parts, among them J101 SOLDER_JUMPER_CONN, J102 SOLDER_JUMPER_CONN, J103 SOLDER_JUMPER_CONN, J104 RJ12, J105 RJ12, P101 CONN_01X02, P102 CONN_01X04, P103 CONN_01X05, Q101 BC857, Q102 BC849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

Commit message: Small cleanups
Parts:
- removed C101: CAP, Capacitors_SMD:c_elec_5x4.5
- removed D103: D_Small, Diodes_SMD:Diode-Universal-SMA-SMB_Handsoldering
- removed REF**: MountingHole_3mm, Mounting_Holes:MountingHole_3mm
- removed REF** (x2): Mousebite, Other:Mousebite
- removed REF**: Symbol_OSHW-Logo_SilkScreen, Symbols:Symbol_OSHW-Logo_SilkScreen
- removed U104: LM1117, Kicad_Library:SOT-223
- added C102: 330uF, Capacitors_SMD:CP_Elec_10x10, F.Cu at (194.3, 155.8)
- added C103: 330uF, Capacitors_SMD:CP_Elec_10x10, F.Cu at (210.3, 156.5)
- added D105: DF01S, pyth:DIPSMD4, F.Cu at (182.7, 145.7)
- added D106: 1N5821, kicad-libraries:DO-214AA, F.Cu at (195.9, 142.0)
- added JP101: JUMPER3, Other:SolderJumper2way, F.Cu at (204.0, 135.5)
- added U111: LM2575-5, TO_SOT_Packages_SMD:TO-263-5Lead, F.Cu at (238.6, 144.0)
- J101, J102, J103: footprint Other:solder_jumper_conn -> kicad-libraries:SolderJumper
- moved U110 18.5 mm to (183.0, 79.6)
Connections:
- net ack renamed ACK
- J104 pad 2: DC_GND -> GND
- J104 pad 5: DC_GND -> GND
- J105 pad 2: DC_GND -> GND
- J105 pad 5: DC_GND -> GND
- P102 pad 4: DC_GND -> GND
- Q102 pad 2: DC_GND -> GND
- R111 pad 2: DC_GND -> GND
- R113 pad 2: DC_GND -> GND
- U101 pad 2: DC_GND -> GND
- U101 pad 4: DC_GND -> GND
- U101 pad 6: DC_GND -> GND
- U101 pad 8: DC_GND -> GND
- U102 pad 5: DC_GND -> GND
- U103 pad 1: DC_GND -> GND
- U105 pad 10: DC_GND -> GND
- U105 pad 14: DC_GND -> GND
- U105 pad 2: Loconet_RX -> Net-(JP101-Pad1)
- U105 pad 6: Loconet_RX -> Net-(JP101-Pad3)
- U105 pad 9: DC_GND -> GND
- U106 pad 1: DC_GND -> GND
- U106 pad 4: DC_GND -> GND
Routing:
- net DC_GND: track 170.5 -> 0.00 mm, vias 16 -> 0
- net Track_O: track 124.8 -> 0.00 mm
- net Track_B: track 116.7 -> 0.00 mm, vias 2 -> 0
- net VCC: track 102.9 -> 0.00 mm, vias 4 -> 0
- net Loconet_RX: track 79.8 -> 0.00 mm
- net tracksignal: track 53.6 -> 0.00 mm
- net Loconet_TX: track 46.3 -> 0.00 mm
- net Loconet: track 41.9 -> 0.00 mm
- net DC_PLUS: track 34.8 -> 0.00 mm
- net Net-(D101-Pad1): track 27.0 -> 0.00 mm
- net Net-(R110-Pad2): track 20.4 -> 0.00 mm
- net FBO1: track 19.5 -> 0.00 mm
- net FBO_COMMON: track 18.6 -> 0.00 mm
- net Net-(R112-Pad2): track 16.8 -> 0.00 mm
- net FBO2: track 15.9 -> 0.00 mm
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- removed copper zone on B.Cu, net DC_GND
- removed copper zone on F.Cu, net DC_GND
Other:
- outline, holes or cut-outs redrawn
