File: 3016_21mtc/3016_21mtc.kicad_pcb (KiCad board)
At the start: 2 copper layers, 60 x 19 mm, 33 parts, among them P1 CONN_01X01, P10 CONN_01X01, P102 CONN_02X11, P11 CONN_01X01, P12 CONN_01X01, P13 CONN_01X01, P14 CONN_01X01, P15 CONN_01X01, P16 CONN_01X01, P17 CONN_01X01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

Commit message: Added gerbers
Other:
- board text added: "3016 board, Rev.0 https://github.com/dirkjankrijnders/decint J.D. Krijnders, 2017-06-13"
Changed lines of the file:
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@@
     (area 94.870199 64.620199 161.042896 85.4298)
     (thickness 1.6)
-    (drawings 15)
+    (drawings 16)
     (tracks 466)
     (zones 0)
@@
       (xy 1.951567 0.478367)) (layer F.SilkS) (width 0.001))
   )
+  (gr_text "3016 board, Rev.0\nhttps://github.com/dirkjankrijnders/decint\nJ.D. Krijnders, 2017-06-13" (at 103.2002 76.6318 180) (layer B.SilkS)
+    (effects (font (size 1 1) (thickness 0.2)) (justify left mirror))
+  )
   (gr_text "F R 4 3 2 1 5 H3" (at 109.22 71.5518) (layer F.SilkS)
